File: Hardware/Motherboard/TinyTendo.kicad_pcb (KiCad board)
At the start: 4 copper layers, 64.7 x 52.2 mm, 51 parts, among them J1 Conn_01x01_Male, J2 Conn_01x01_Male, J3 Conn_01x01_Male, J4 Conn_01x01_Male, J5 Conn_01x01_Male, J6 Conn_01x01_Male, J7 Conn_01x01_Male, J8 Conn_01x01_Male, J9 Conn_01x01_Male, P1 72-Pin Connector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

Commit message: Initial Commit
Initial layout using original IC's with no cuts.
Parts:
- C1, C10, C2, C3, C4, C5, C6, C8, C9, L1, R1, R2, R3, R4, R5, R6, R7, R8, U3, U4, U5, U6, U7, X1: moved to B.Cu
- U1, U2: footprint TinyTendo:Cut chip -> Package_DIP:DIP-40_W15.24mm
- moved J4 60.1 mm to (176.7, 85.3)
- moved J6 60.1 mm to (176.6, 87.7)
- moved J5 60.0 mm to (176.7, 82.9)
- moved J7 58.6 mm to (176.5, 95.9)
- moved J8 58.6 mm to (176.5, 98.4)
- moved C9 48.6 mm to (182.0, 90.9)
- moved L1 48.3 mm to (182.0, 92.8)
- moved C7 47.9 mm to (181.5, 81.0), turned to 0 degrees
- moved R1 46.1 mm to (179.2, 96.2)
- moved C8 45.3 mm to (185.0, 91.9), turned to -90 degrees
- moved R4 44.0 mm to (183.3, 96.2)
- moved R3 44.0 mm to (181.3, 96.2)
- moved R2 42.2 mm to (185.3, 96.2)
- moved C10 42.0 mm to (187.7, 113.4)
- moved U2 35.7 mm to (178.8, 99.9), turned to 90 degrees
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Connections:
- net /CPU-R~W renamed /CPU-R~{W}
- net /PPU-~A13 renamed /PPU-~{A13}
- net /PPU-~CE renamed /PPU-~{CE}
- net /PPU-~RD renamed /PPU-~{RD}
- net /PPU-~WE renamed /PPU-~{WE}
- net /VRAM-~CE renamed /VRAM-~{CE}
- net /WRAM-~CE renamed /WRAM-~{CE}
- net /~IRQ renamed /~{IRQ}
- net /~NMI renamed /~{NMI}
- net /~OE1 renamed /~{OE1}
- net /~OE2 renamed /~{OE2}
- net /~ROMSEL renamed /~{ROMSEL}
- net /~RST renamed /~{RST}
Routing:
- net /CPU-A5: track 34.7 -> 97.2 mm, vias 0 -> 1
- net /CPU-A3: track 36.2 -> 97.7 mm, vias 0 -> 1
- net /CPU-A4: track 33.8 -> 93.8 mm, vias 0 -> 1
- net /CPU-A7: track 33.3 -> 86.9 mm, vias 0 -> 1
- net /CPU-A6: track 34.2 -> 84.9 mm, vias 0 -> 1
- net /SYS-CLK: track 34.2 -> 84.4 mm, vias 0 -> 2
- net /PPU-A7: track 27.7 -> 75.6 mm, vias 2 -> 3
- net /PPU-~{CE}: track 31.5 -> 79.3 mm, vias 2 -> 0
- net /~{NMI}: track 30.7 -> 69.5 mm, vias 0 -> 1
- net /M2: track 63.0 -> 100.6 mm, vias 4 -> 2
- net /OUT-0: track 39.8 -> 6.23 mm, vias 2 -> 1
- net /PPU-D7: track 52.9 -> 85.6 mm, vias 3 -> 1
- net /CPU-A8: track 44.2 -> 76.7 mm, vias 3 -> 1
- net /CPU-R~{W}: track 66.0 -> 97.5 mm, vias 5 -> 1
- net /CPU-A1: track 54.6 -> 85.8 mm, vias 4 -> 1
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- removed copper zone on F.Cu, net /3V3
Other:
- net class Default removed
- board text removed: "= DIP Pin 1"
- board text removed: "Must be 10x10mm"
